File: HoverboardPCBElectricSchematic/TAOTAO TT-SD2.2.sch (EAGLE design)
At the start: 54 parts, among them Q3 BC849, Q4 BC849, Q5 BC849, Q6 BC849, Q7 BC849, U1 7805DT, U16 7805DT

Commit message: Add files via upload
Parts:
- added C3: (no value), rcl:C-EU025-025X050
Connections:
- net GND: now also C3.2
- net N$58: now also C3.1
Changed lines of the file:
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@@
 <part name="R52" library="rcl" library_urn="urn:adsk.eagle:library:334" deviceset="R-EU_" device="0207/2V" package3d_urn="urn:adsk.eagle:package:23490/1" value="1K"/>
 <part name="GND4" library="supply1" library_urn="urn:adsk.eagle:library:371" deviceset="GND" device=""/>
+<part name="C3" library="rcl" library_urn="urn:adsk.eagle:library:334" deviceset="C-EU" device="025-025X050" package3d_urn="urn:adsk.eagle:package:23629/1"/>
 </parts>
 <sheets>
@@
 <attribute name="VALUE" x="125.69" y="41.198" size="1.778" layer="96"/>
 </instance>
+<instance part="C3" gate="G$1" x="166" y="49" smashed="yes">
+<attribute name="NAME" x="167.524" y="49.381" size="1.778" layer="95"/>
+<attribute name="VALUE" x="167.524" y="44.301" size="1.778" layer="96"/>
+</instance>
 </instances>
 <busses>
@@
 <pinref part="GND20" gate="1" pin="GND"/>
 <wire x1="141.5" y1="42.42" x2="141.5" y2="37.54" width="0.1524" layer="91"/>
+<pinref part="C3" gate="G$1" pin="2"/>
+<wire x1="166" y1="43.92" x2="166" y2="37.54" width="0.1524" layer="91"/>
+<wire x1="166" y1="37.54" x2="141.5" y2="37.54" width="0.1524" layer="91"/>
+<junction x="141.5" y="37.54"/>
 </segment>
 </net>
@@
 <pinref part="R67" gate="G$1" pin="2"/>
 <wire x1="141.5" y1="64.58" x2="141.5" y2="66.96" width="0.1524" layer="91"/>
-</segment>
-</net>
+<pinref part="C3" gate="G$1" pin="1"/>
+<wire x1="166" y1="51.54" x2="166" y2="64.58" width="0.1524" layer="91"/>
+<wire x1="166" y1="64.58" x2="141.5" y2="64.58" width="0.1524" layer="91"/>
+<junction x="141.5" y="64.58"/>
+</segment>
+</net>
